File: KICAD/RCMhardwareV4.kicad_pcb (KiCad board)
At the start: 2 copper layers, 50.8 x 76.2 mm, 39 parts, among them J1 Conn_01x05_Pin, J10 Conn_01x04_Pin, J11 Conn_01x04_Pin, J12 Conn_01x02_Pin, J13 Conn_01x02_Pin, J14 Conn_01x02_Pin, J15 Conn_01x02_Pin, J16 Conn_01x02_Pin, J17 Conn_02x03_Odd_Even, J2 Conn_01x02_Pin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

Commit message: Update RCMhardwareV4.kicad_pcb
Other:
- board text added: "RCMV4 v1.0"
- board text removed: "RCMv4.0.0"
Changed lines of the file:
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@@
     (effects (font (size 1 1) (thickness 0.15)) (justify left bottom mirror))
   )
-  (gr_text "RCMv4.0.0" (at 77.6732 126.1364) (layer "B.SilkS")
+  (gr_text "RCMV4  v1.0" (at 78.232 125.73) (layer "B.SilkS")
     (effects (font (size 1 1) (thickness 0.15)) (justify left bottom mirror))
   )

Commit message: v1.1.1
Parts:
- TP2: moved to B.Cu
- turned TP2 to 180 degrees
Routing:
- net IC3 2A: track 102.5 -> 101.3 mm
Other:
- board text added: "+ -"
- board text added: "21 22"
- board text added: "G 3v 3 2 1"
- board text added: "RCMV4 v1.1"
- board text added: "inport"
- board text added: "v1.1"
- board text removed: "RCMV4 v1.0"

Commit message: v1.2 close #3 #4 #5
Parts:
- R2, R3: footprint Resistor_THT:R_Axial_DIN0204_L3.6mm_D1.6mm_P7.62mm_Horizontal -> Resistor_THT:R_Axial_DIN0207_L6.3mm_D2.5mm_P10.16mm_Horizontal
- moved R3 1.31 mm to (81.9, 93.9)
- moved J13 1.27 mm to (55.9, 86.4)
- moved J14 1.27 mm to (55.9, 91.4)
- moved J15 1.27 mm to (55.9, 106.7)
- moved J16 1.27 mm to (55.9, 111.8)
Routing:
- net IC3 1B: track 88.6 -> 116.1 mm, vias 4 -> 3
- net vbat: track 212.9 -> 187.6 mm, vias 0 -> 2
- net Net-(J12-Pin_1): track 49.8 -> 37.3 mm
- net IC3 2B: track 55.6 -> 50.2 mm
- net Net-(J13-Pin_2): track 29.4 -> 31.4 mm
- net sda: track 79.6 -> 77.8 mm
- net Net-(J12-Pin_2): track 30.7 -> 32.2 mm
- net Net-(J13-Pin_1): track 35.2 -> 36.7 mm
- net IC3 1A: track 43.9 -> 45.2 mm
- net Net-(U1-SENSOR_VP): track 10.1 -> 8.84 mm
- net IC1 1B: track 15.7 -> 14.6 mm
- net IC3 2A: track 101.3 -> 100.3 mm
- net Net-(J2-Pin_1): track 28.2 -> 27.5 mm
- net Net-(J14-Pin_1): track 45.7 -> 46.3 mm
- net Net-(J16-Pin_1): track 24.0 -> 24.5 mm
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Other:
- board text added: "3 2 1"
- board text added: "7 6 5 4"
- board text added: "RCMV4 v1.2"
- board text added: "v1.2"
- board text removed: "7 6 5 4 3 2 1"
- board text removed: "RCMV4 v1.1"
- board text removed: "v1.1"

Commit message: v1.3
Parts:
- J3, J4, J5, J6: footprint Connector_PinHeader_2.54mm:PinHeader_1x07_P2.54mm_Vertical -> projectlib:PinHeader_1x07_P2.54mm_Vertical
- moved J12 2.54 mm to (55.9, 104.1), turned to 180 degrees
- moved J13 2.54 mm to (55.9, 88.9), turned to 180 degrees
- moved J14 2.54 mm to (55.9, 94.0), turned to 180 degrees
- moved J2 2.54 mm to (55.9, 99.1), turned to 180 degrees
- moved J15 2.54 mm to (55.9, 109.2), turned to 180 degrees
- moved J16 2.54 mm to (55.9, 114.3), turned to 180 degrees
- moved J9 0.51 mm to (97.2, 103.9)
- moved J10 0.51 mm to (97.2, 113.0)
Connections:
- U2 pad 11: Net-(J12-Pin_2) -> Net-(J12-Pin_1)
- U2 pad 14: Net-(J12-Pin_1) -> Net-(J12-Pin_2)
- U2 pad 3: Net-(J2-Pin_1) -> Net-(J2-Pin_2)
- U2 pad 6: Net-(J2-Pin_2) -> Net-(J2-Pin_1)
- U3 pad 11: Net-(J14-Pin_2) -> Net-(J14-Pin_1)
- U3 pad 14: Net-(J14-Pin_1) -> Net-(J14-Pin_2)
- U3 pad 3: Net-(J13-Pin_1) -> Net-(J13-Pin_2)
- U3 pad 6: Net-(J13-Pin_2) -> Net-(J13-Pin_1)
- U4 pad 11: Net-(J16-Pin_2) -> Net-(J16-Pin_1)
- U4 pad 14: Net-(J16-Pin_1) -> Net-(J16-Pin_2)
- U4 pad 3: Net-(J15-Pin_1) -> Net-(J15-Pin_2)
- U4 pad 6: Net-(J15-Pin_2) -> Net-(J15-Pin_1)
Routing:
- net Net-(J16-Pin_2): track 15.9 -> 24.5 mm
- net Net-(J16-Pin_1): track 24.5 -> 15.9 mm
- net Net-(J15-Pin_2): track 14.8 -> 23.5 mm
- net Net-(J15-Pin_1): track 23.5 -> 14.8 mm
- net Net-(J14-Pin_2): track 41.0 -> 46.3 mm
- net Net-(J13-Pin_2): track 31.4 -> 36.7 mm
- net Net-(J13-Pin_1): track 36.7 -> 31.4 mm
- net Net-(J12-Pin_2): track 32.2 -> 37.3 mm
- net Net-(J12-Pin_1): track 37.3 -> 32.2 mm
- net Net-(J14-Pin_1): track 46.3 -> 41.6 mm
- net Net-(J2-Pin_2): track 24.1 -> 27.5 mm, vias 0 -> 2
- net Net-(J2-Pin_1): track 27.5 -> 24.1 mm, vias 2 -> 0
- net GND: track 17.9 -> 18.7 mm
- net vbat: track 187.6 -> 188.3 mm
- net +3.3V: track 71.2 -> 71.9 mm
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Other:
- board text added: "RCMV4 v1.3"
- board text added: "esp usb"
- board text added: "v1.3"
- board text removed: "RCMV4 v1.2"
- board text removed: "v1.2"
