File: KICAD/RCMhardwareV4.kicad_sch (KiCad schematic)
At the start: 33 parts, among them J1 Conn_01x05_Pin, J10 Conn_01x04_Pin, J11 Conn_01x04_Pin, J12 Conn_01x02_Pin, J13 Conn_01x02_Pin, J14 Conn_01x02_Pin, J15 Conn_01x02_Pin, J16 Conn_01x02_Pin, J17 Conn_02x03_Odd_Even, J2 Conn_01x02_Pin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

Commit message: v1.1.1
Other:
- note added: "22 21"
- note added: "ESP 5V"
- note added: "L293D #1"
- note added: "L293D #2"
- note added: "L293D #3"
- note added: "servo pwr"
- company: (none) -> RCMGames
- title: (none) -> RCM V4
Changed lines of the file:
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@@
 (kicad_sch (version 20230121) (generator eeschema)
   (paper "A4")
+  (title_block
+    (title "RCM V4")
+    (rev "v1.1")
+    (company "RCMGames")
+  )
   (junction (at 44.45 63.5) (diameter 0) (color 0 0 0 0)
   )
@@
     (effects (font (size 1.27 1.27)) (justify left bottom))
   )
+  (text "L293D #3\n" (at 71.12 135.89 0)
+    (effects (font (size 1.27 1.27)) (justify left bottom))
+  )
+  (text "servo pwr\n" (at 223.52 62.23 0)
+    (effects (font (size 1.27 1.27)) (justify left bottom))
+  )
   (text "for soldering practice\nor tiny prototyping" (at 207.01 38.1 0)
     (effects (font (size 1.27 1.27)) (justify left bottom))
   )
   (text "RSL\n" (at 167.64 72.39 0)
+    (effects (font (size 1.27 1.27)) (justify left bottom))
+  )
+  (text "L293D #2\n" (at 62.23 77.47 0)
+    (effects (font (size 1.27 1.27)) (justify left bottom))
+  )
+  (text "22\n21\n" (at 269.24 22.86 0)
+    (effects (font (size 1.27 1.27)) (justify left bottom))
+  )
+  (text "ESP 5V" (at 133.35 104.14 0)
     (effects (font (size 1.27 1.27)) (justify left bottom))
   )
@@
   )
   (text "reset" (at 120.65 39.37 0)
+    (effects (font (size 1.27 1.27)) (justify left bottom))
+  )
+  (text "L293D #1\n" (at 60.96 20.32 0)
     (effects (font (size 1.27 1.27)) (justify left bottom))
   )
@@
   )
   (symbol (lib_id "Connector:Conn_01x04_Pin") (at 267.97 25.4 180) (unit 1)
-    (in_bom yes) (on_board yes) (dnp no) (fields_autoplaced)
-    (property "Reference" "J11" (at 269.24 22.86 0)
+    (in_bom yes) (on_board yes) (dnp no)
+    (property "Reference" "J11" (at 269.24 25.4 0)
       (effects (font (size 1.27 1.27)) (justify right))
     )
-    (property "Value" "Conn_01x04_Pin" (at 269.24 25.4 0)
+    (property "Value" "Conn_01x04_Pin" (at 269.24 27.94 0)
       (effects (font (size 1.27 1.27)) (justify right))
     )

Commit message: v1.2 close #3 #4 #5
Parts:
- R2, R3: footprint Resistor_THT:R_Axial_DIN0204_L3.6mm_D1.6mm_P7.62mm_Horizontal -> Resistor_THT:R_Axial_DIN0207_L6.3mm_D2.5mm_P10.16mm_Horizontal
Other:
- note removed: "can't be pulled high on boot, but could work for motor?"
- note removed: "pullup, use for servo"
- note removed: "weak pullup, but no pwm detected, test for servo pin"
Changed lines of the file:
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@@
   (title_block
     (title "RCM V4")
-    (rev "v1.1")
+    (rev "v1.2")
     (company "RCMGames")
   )
@@
     (stroke (width 0) (type default))
   )
-  (text "weak pullup, but no pwm detected, test for servo pin"
-    (at 73.66 63.5 0)
-    (effects (font (size 1.27 1.27)) (justify left bottom))
-  )
   (text "in only" (at 124.46 48.26 90)
     (effects (font (size 1.27 1.27)) (justify left bottom))
@@
     (effects (font (size 1.27 1.27)) (justify left bottom))
   )
-  (text "can't be pulled high on boot, but could work for motor?"
-    (at 62.23 68.58 0)
-    (effects (font (size 1.27 1.27)) (justify left bottom))
-  )
   (text "reset" (at 120.65 39.37 0)
     (effects (font (size 1.27 1.27)) (justify left bottom))
@@
   )
   (text "IO 0\n" (at 170.18 69.85 0)
-    (effects (font (size 1.27 1.27)) (justify left bottom))
-  )
-  (text "pullup, use for servo" (at 177.8 59.69 0)
     (effects (font (size 1.27 1.27)) (justify left bottom))
   )
@@
       (effects (font (size 1.27 1.27)))
     )
-    (property "Footprint" "Resistor_THT:R_Axial_DIN0204_L3.6mm_D1.6mm_P7.62mm_Horizontal" (at 107.95 27.432 90)
+    (property "Footprint" "Resistor_THT:R_Axial_DIN0207_L6.3mm_D2.5mm_P10.16mm_Horizontal" (at 107.95 27.432 90)
       (effects (font (size 1.27 1.27)) hide)
     )
@@
       (effects (font (size 1.27 1.27)))
     )
-    (property "Footprint" "Resistor_THT:R_Axial_DIN0204_L3.6mm_D1.6mm_P7.62mm_Horizontal" (at 115.57 27.432 90)
-      (effects (font (size 1.27 1.27)) hide)
-    )
+    (property "Footprint" "Resistor_THT:R_Axial_DIN0207_L6.3mm_D2.5mm_P10.16mm_Horizontal" (at 115.57 27.432 90)
+      (effects (font (size 1.27 1.27)) hide)
+    )

Commit message: v1.3
Parts:
- J3, J4, J5, J6: footprint Connector_PinHeader_2.54mm:PinHeader_1x07_P2.54mm_Vertical -> projectlib:PinHeader_1x07_P2.54mm_Vertical
Connections:
- net at J16.1 (Pin_1): now also U4.11 (3Y); no longer U4.14 (4Y)
- net at J16.2 (Pin_2): now also U4.14 (4Y); no longer U4.11 (3Y)
- net at U2.11 (3Y): now also J12.1 (Pin_1); no longer J12.2 (Pin_2)
- net at U2.14 (4Y): now also J12.2 (Pin_2); no longer J12.1 (Pin_1)
- net at U2.3 (1Y): now also J2.2 (Pin_2); no longer J2.1 (Pin_1)
- net at U2.6 (2Y): now also J2.1 (Pin_1); no longer J2.2 (Pin_2)
- net at U4.3 (1Y): now also J15.2 (Pin_2); no longer J15.1 (Pin_1)
- net at U4.6 (2Y): now also J15.1 (Pin_1); no longer J15.2 (Pin_2)
- net at U3.11 (3Y): now also J14.1 (Pin_1); no longer J14.2 (Pin_2)
- net at U3.14 (4Y): now also J14.2 (Pin_2); no longer J14.1 (Pin_1)
- net at U3.3 (1Y): now also J13.2 (Pin_2); no longer J13.1 (Pin_1)
- net at U3.6 (2Y): now also J13.1 (Pin_1); no longer J13.2 (Pin_2)
